Commit message: feat(description): urdf raspi pi camera module and zed x mini stero camera added

File: urdf/camera.xacro (robot description, xacro)
@@ -4,28 +4,30 @@
     <xacro:include filename="$(find waver_description)/urdf/util.xacro" />
     <link name="camera_link">
+        <inertial>
+            <mass value="${rasp_pi_camera_mass}" />
+            <origin xyz="0 0 0" rpy="0 0 0" />
+            <inertia ixx="8.188544198245058e-07" iyy="1.3934609636775025e-06" izz="8.837267894803364e-07" ixy="0" iyz="0" ixz="0" />
+        </inertial>
+        <visual>
+            <origin xyz="0 0.0125 0" rpy="0 0 ${-pi/2}" />
+            <geometry>
+                <mesh filename="file:///$(find waver_description)/meshes/rasp_pi_camera.stl" scale="${camera_scale}" />
+            </geometry>
+            <xacro:black_material />
+        </visual>
         <collision>
-            <origin xyz="0 0 0" rpy="0 0 0"/>
+            <origin xyz="0 0.0125 0" rpy="0 0 ${-pi/2}" />
             <geometry>
-                <box size="0.003 0.015 0.015"/>
+                <mesh filename="file:///$(find waver_description)/meshes/rasp_pi_camera.stl" scale="${camera_scale}" />
             </geometry>
         </collision>
-        <visual>
-            <origin xyz="0 0 0" rpy="0 0 0"/>
-            <geometry>
-                <box size="0.003 0.015 0.015"/>
-            </geometry>
-        </visual>
-        <inertial>
-            <mass value="0.0001" />
-            <origin xyz="0 0 0" rpy="0 0 ${pi}"/>
-            <inertia ixx="0.0000001" ixy="0" ixz="0" iyy="0.0000001" iyz="0" izz="0.0000001" />
-        </inertial>
     </link>
     <joint name="camera_sensor_joint" type="fixed">
-        <origin xyz="0.06 0 0.065" rpy="0 0 0"/>
-        <parent link="top_shell_link"/>
-        <child link="camera_link"/>
+        <origin xyz="0.09 0 ${base_to_top}" rpy="0 0 0" />
+        <parent link="top_shell_link" />
+        <child link="camera_link" />
     </joint>
     <gazebo reference="camera_link">
+        <material>Gazebo/Black</material>
         <sensor type="camera" name="camera">
             <update_rate>30.0</update_rate>

File: urdf/util.xacro (robot description, xacro)
@@ -100,3 +100,9 @@
     <xacro:property name="lidar_frequency" value="10" />
     <xacro:property name="lidar_transform" value="0 0 0 0 0 0" />
+    <!-- Rasp Pi Camera specifications -->
+    <xacro:property name="rasp_pi_camera_mass" value="0.0035" />
+    <xacro:property name="camera_scale" value="0.0005 0.0005 0.0005" />
+    <!-- ZED X Mini Stereo Camera specifications -->
+    <xacro:property name="zed_x_mini_mass" value="0.015" />
+    <xacro:property name="zed_x_mini_scale" value="1 1 1" />
 </robot>

File: urdf/waver.xacro (robot description, xacro)
@@ -1,4 +1,5 @@
 <?xml version="1.0"?>
 <robot name="waver" xmlns:xacro="http://www.ros.org/wiki/xacro">
+  <xacro:arg name="camera_type" default="raspi" />
   <xacro:include filename="$(find waver_description)/urdf/materials.xacro" />
   <xacro:include filename="$(find waver_description)/urdf/util.xacro" />
@@ -7,5 +8,10 @@
   <xacro:include filename="$(find waver_description)/urdf/lidar.xacro" />
   <xacro:include filename="$(find waver_description)/urdf/imu.xacro" />
-  <xacro:include filename="$(find waver_description)/urdf/camera.xacro" />
+  <xacro:if value="${'$(arg camera_type)' == 'raspi'}">
+    <xacro:include filename="$(find waver_description)/urdf/camera.xacro" />
+  </xacro:if>
+  <xacro:if value="${'$(arg camera_type)' == 'depth'}">
+    <xacro:include filename="$(find waver_description)/urdf/depth_camera.xacro" />
+  </xacro:if>
   <!-- ******************************* Links ******************************* -->
   <link name="base_footprint"></link>
