Commit message: feat(descr): gz sim new version implementation

File: urdf/camera.xacro (robot description, xacro)
@@ -4,9 +4,4 @@
     <xacro:include filename="$(find waver_description)/urdf/util.xacro" />
     <link name="camera_link">
-        <inertial>
-            <mass value="${rasp_pi_camera_mass}" />
-            <origin xyz="0 0 0" rpy="0 0 0" />
-            <inertia ixx="8.188544198245058e-07" iyy="1.3934609636775025e-06" izz="8.837267894803364e-07" ixy="0" iyz="0" ixz="0" />
-        </inertial>
         <visual>
             <origin xyz="0 0.0125 0" rpy="0 0 ${-pi/2}" />
@@ -17,7 +12,7 @@
         </visual>
         <collision>
-            <origin xyz="0 0.0125 0" rpy="0 0 ${-pi/2}" />
+            <origin xyz="0.005 0 -0.012" rpy="0 0 0" />
             <geometry>
-                <mesh filename="file:///$(find waver_description)/meshes/rasp_pi_camera.stl" scale="${camera_scale}" />
+                <box size="0.01 0.025 0.023" />
             </geometry>
         </collision>
@@ -30,16 +25,19 @@
     <gazebo reference="camera_link">
         <material>Gazebo/Black</material>
-        <sensor type="camera" name="camera">
-            <update_rate>30.0</update_rate>
-            <camera name="head">
-                <horizontal_fov>1.3962634</horizontal_fov>
+        <sensor name="camera" type="camera">
+            <pose>0 0 -0.0135 0 0 0</pose>
+            <visualize>false</visualize>
+            <update_rate>30</update_rate>
+            <topic>camera</topic>
+            <camera>
+                <horizontal_fov>1.1519</horizontal_fov>
                 <image>
-                    <width>800</width>
-                    <height>600</height>
                     <format>R8G8B8</format>
+                    <height>1080</height>
+                    <width>1920</width>
                 </image>
                 <clip>
-                    <near>0.02</near>
-                    <far>300</far>
+                    <near>0.10</near>
+                    <far>100.0</far>
                 </clip>
                 <noise>
@@ -49,18 +47,4 @@
                 </noise>
             </camera>
-            <plugin name="camera_controller" filename="libgazebo_ros_camera.so">
-                <alwaysOn>true</alwaysOn>
-                <updateRate>0.0</updateRate>
-                <cameraName>iRobot/camera</cameraName>
-                <imageTopicName>image_raw</imageTopicName>
-                <cameraInfoTopicName>camera_info</cameraInfoTopicName>
-                <frameName>camera_link</frameName>
-                <hackBaseline>0.07</hackBaseline>
-                <distortionK1>0.0</distortionK1>
-                <distortionK2>0.0</distortionK2>
-                <distortionK3>0.0</distortionK3>
-                <distortionT1>0.0</distortionT1>
-                <distortionT2>0.0</distortionT2>
-            </plugin>
         </sensor>
     </gazebo>

File: urdf/depth_camera.xacro (robot description, xacro)
@@ -4,10 +4,4 @@
     <xacro:include filename="$(find waver_description)/urdf/util.xacro" />
     <link name="camera_link">
-        <inertial>
-            <mass value="${zed_x_mini_mass}" />
-            <origin xyz="0 0 0" rpy="0 0 0" />
-            <inertia ixx="1.2205537500280872e-05" iyy="4.073932956405751e-06"
-                izz="1.3748504884318975e-05" ixy="0" iyz="0" ixz="0" />
-        </inertial>
         <visual>
             <origin xyz="0 0 0" rpy="0 0 0" />
@@ -19,8 +13,7 @@
         </visual>
         <collision>
-            <origin xyz="0 0 0" rpy="0 0 0" />
+            <origin xyz="0 0 ${base_to_top - 0.039}" rpy="0 0 0" />
             <geometry>
-                <mesh filename="file:///$(find waver_description)/meshes/zedxm.stl"
-                    scale="${zed_x_mini_scale}" />
+                <box size="${zed_x_mini_dimensions}" />
             </geometry>
         </collision>
@@ -39,7 +32,9 @@
     <gazebo reference="camera_link">
         <material>Gazebo/Black</material>
-        <sensor name="camera" type="depth">
+        <sensor name="depth_camera" type="rgbd_camera">
             <visualize>true</visualize>
-            <update_rate>60.0</update_rate>
+            <update_rate>30.0</update_rate>
+            <topic>depth_camera</topic>
+            <gz_frame_id>camera_link</gz_frame_id>
             <camera>
                 <horizontal_fov>1.047198</horizontal_fov>
@@ -59,22 +54,4 @@
                 </noise>
             </camera>
-            <plugin name="depth_camera_controller" filename="libgazebo_ros_camera.so">
-                <baseline>0.05</baseline>
-                <alwaysOn>true</alwaysOn>
-                <updateRate>60.0</updateRate>
-                <frame_name>camera_optical_frame</frame_name>
-                <pointCloudCutoff>0.1</pointCloudCutoff>
-                <pointCloudCutoffMax>8.0</pointCloudCutoffMax>
-                <distortionK1>0</distortionK1>
-                <distortionK2>0</distortionK2>
-                <distortionK3>0</distortionK3>
-                <distortionT1>0</distortionT1>
-                <distortionT2>0</distortionT2>
-                <CxPrime>0</CxPrime>
-                <Cx>0</Cx>
-                <Cy>0</Cy>
-                <focalLength>0</focalLength>
-                <hackBaseline>0</hackBaseline>
-            </plugin>
         </sensor>
     </gazebo>

File: urdf/imu.xacro (robot description, xacro)
@@ -4,9 +4,4 @@
     <xacro:include filename="$(find waver_description)/urdf/util.xacro" />
     <link name="imu_link">
-        <inertial>
-            <mass value="${mass_imu}" />
-            <origin xyz="${mass_center_imu}" rpy="0 0 ${pi/2}" />
-            <inertia ixx="4.297064285474092e-13" iyy="4.199442581059605e-13" izz="7.142756866533696e-13" ixy="0.0" iyz="0.0" ixz="0.0" />
-        </inertial>
         <visual>
             <origin xyz="${position_imu}" rpy="0 0 ${pi/2}" />
@@ -16,10 +11,4 @@
             <xacro:dark_green_material />
         </visual>
-        <collision>
-            <origin xyz="${position_imu}" rpy="0 0 ${pi/2}" />
-            <geometry>
-                <mesh filename="file:///$(find waver_description)/meshes/board_link.stl" scale="${scale}" />
-            </geometry>
-        </collision>
     </link>
     <joint name="top_imu_joint" type="fixed">
@@ -29,34 +18,11 @@
     </joint>
     <gazebo reference="imu_link">
-        <!-- <sensor name="imu_sensor" type="imu">
+        <material>Gazebo/Orange</material>
+        <gravity>true</gravity>
+        <sensor name="imu_sensor" type="imu">
             <always_on>true</always_on>
             <update_rate>100</update_rate>
             <visualize>true</visualize>
-            <plugin filename="libgazebo_ros_imu_sensor.so" name="gazebo_ros_imu_sensor">
-                <ros>
-                    <namespace></namespace>
-                    <remapping>imu:=imu/data_raw</remapping>
-                </ros>
-                <frame_name>imu_link</frame_name>
-                <update_rate>100.0</update_rate>
-                <orientation_reference_frame>world</orientation_reference_frame>
-                <imu_parameters>
-                    <noise_density>0.0025</noise_density>
-                    <bias_correlation_time>1000000.0</bias_correlation_time>
-                    <random_walk>0.0002</random_walk>
-                </imu_parameters>
-            </plugin>
-        </sensor> -->
-        <sensor name="imu_sensor" type="imu">
-        <!-- ensure the sensor is active (required) -->
-        <always_on>true</always_on>
-        <update_rate>50</update_rate>
-        <plugin name="my_imu_plugin" filename="libgazebo_ros_imu_sensor.so">
-            <ros>
-            <!-- publish to /imu/data -->
-            <namespace>/imu</namespace>
-            <remapping>~/out:=data</remapping>
-            </ros>
-        </plugin>
+            <topic>imu</topic>
         </sensor>
     </gazebo>

File: urdf/lidar.xacro (robot description, xacro)
@@ -3,5 +3,5 @@
     <xacro:include filename="$(find waver_description)/urdf/materials.xacro" />
     <xacro:include filename="$(find waver_description)/urdf/util.xacro" />
-    <link name="${lidar_link}">
+    <link name="lidar_link">
         <inertial>
             <mass value="${mass_lidar}" />
@@ -17,7 +17,7 @@
         </visual>
         <collision>
-            <origin xyz="0 0 -0.027" rpy="0 0 ${pi/2}" />
+            <origin xyz="0 0 -0.0107" rpy="0 0 0" />
             <geometry>
-                <mesh filename="file:///$(find waver_description)/meshes/LD19.stl" scale="${scale}" />
+                <box size="0.0383 0.0383 0.030" />
             </geometry>
         </collision>
@@ -26,12 +26,13 @@
         <origin xyz="0.04 0 ${base_to_top + 0.025}" rpy="0 0 0" />
         <parent link="top_shell_link" />
-        <child link="${lidar_link}" />
+        <child link="lidar_link" />
     </joint>
-    <gazebo reference="${lidar_link}">
+    <gazebo reference="lidar_link">
         <material>Gazebo/Black</material>
-        <sensor name="${lidar_model}" type="ray">
+        <sensor name="lidar_link" type="gpu_lidar">
             <pose>0 0 0 0 0 0</pose>
             <visualize>false</visualize>
             <topic>scan</topic>
+            <gz_frame_id>lidar_link</gz_frame_id>
             <always_on>true</always_on>
             <update_rate>${lidar_frequency}</update_rate>
@@ -48,15 +49,12 @@
                     <min>${lidar_min_range}</min>
                     <max>${lidar_max_range}</max>
+                    <resolution>0.01</resolution>
                 </range>
+                <noise>
+                    <type>gaussian</type>
+                    <mean>0.0</mean>
+                    <stddev>0.01</stddev>
+                </noise>
             </ray>
-            <plugin name="gazebo_ros_laser_controller" filename="libgazebo_ros_ray_sensor.so">
-                <ros>
-                    <!-- Configure namespace and remap to publish to /ray/pointcloud2 -->
-                    <namespace>/</namespace>
-                    <remapping>~/out:=scan</remapping>
-                </ros>
-                <output_type>sensor_msgs/LaserScan</output_type>
-                <frameName>${lidar_link}</frameName>
-            </plugin>
         </sensor>
     </gazebo>

File: urdf/util.xacro (robot description, xacro)
@@ -57,4 +57,5 @@
     <xacro:property name="wheel_separation" value="123e-3" />
     <xacro:property name="wheel_radius" value="40.6e-3" />
+    <xacro:property name="wheel_width" value="42.5e-3" />
     <!-- WBL specifications -->
     <xacro:property name="pos_x_wbl" value="0.06538582611083985" />
@@ -91,6 +92,4 @@
     <!-- Lidar specifications -->
     <xacro:property name="mass_lidar" value="0.046" />
-    <xacro:property name="lidar_model" value="HLS-LFCD-LDS" />
-    <xacro:property name="lidar_link" value="lidar_link" />
     <xacro:property name="lidar_samples" value="720" />
     <xacro:property name="lidar_max_range" value="12.0" />
@@ -106,3 +105,4 @@
     <xacro:property name="zed_x_mini_mass" value="0.015" />
     <xacro:property name="zed_x_mini_scale" value="1 1 1" />
+    <xacro:property name="zed_x_mini_dimensions" value="0.030 0.093 0.0315" />
 </robot>

File: urdf/waver.gazebo.xacro (robot description, xacro)
@@ -62,31 +62,30 @@
     <material>Gazebo/Black</material>
   </gazebo>
-    <gazebo>
-      <plugin name="gazebo_ros_diff_drive" filename="libgazebo_ros_diff_drive.so">
-        <ros>
-          <namespace>/</namespace>
-          <argument>cmd_vel:=cmd_vel</argument>
-        </ros>
-        <always_on>true</always_on>
-        <legacy_mode>true</legacy_mode>
-        <update_rate>50</update_rate>
-        <num_wheel_pairs>2</num_wheel_pairs>
-        <left_joint>wheel_front_left_joint</left_joint>
-        <left_joint>wheel_back_left_joint</left_joint>
-        <right_joint>wheel_front_right_joint</right_joint>
-        <right_joint>wheel_back_right_joint</right_joint>
-        <wheel_separation>${wheel_separation}</wheel_separation>
-        <wheel_diameter>${wheel_radius * 2}</wheel_diameter>
-        <!-- Output -->
-        <odometry_frame>odom</odometry_frame>
-        <odometry_topic>odom</odometry_topic>
-        <robot_base_frame>base_footprint</robot_base_frame>
-        <odometry_source>1</odometry_source>
-        <publish_odom>true</publish_odom>
-        <publish_odom_tf>true</publish_odom_tf>
-        <publish_wheel_tf>true</publish_wheel_tf>
-        <publish_wheel_joint_state>true</publish_wheel_joint_state>
-        <torque>60.0</torque>
-      </plugin>
-    </gazebo>
+  <gazebo>
+    <plugin filename="libgz-sim-diff-drive-system.so" name="gz::sim::systems::DiffDrive">
+      <left_joint>wheel_front_left_joint</left_joint>
+      <right_joint>wheel_front_right_joint</right_joint>
+      <left_joint>wheel_back_left_joint</left_joint>
+      <right_joint>wheel_back_right_joint</right_joint>
+      <wheel_separation>${wheel_separation}</wheel_separation>
+      <wheel_radius>${wheel_radius}</wheel_radius>
+      <max_linear_acceleration>2.0</max_linear_acceleration>
+      <min_linear_acceleration>-2.0</min_linear_acceleration>
+      <max_angular_acceleration>4.0</max_angular_acceleration>
+      <min_angular_acceleration>-4.0</min_angular_acceleration>
+      <topic>cmd_vel</topic>
+      <odom_topic>odometry</odom_topic>
+      <tf_topic>tf</tf_topic>
+      <frame_id>odom</frame_id>
+      <child_frame_id>base_footprint</child_frame_id>
+      <odom_publish_frequency>30</odom_publish_frequency>
+    </plugin>
+    <plugin filename="libgz-sim-joint-state-publisher-system.so"
+      name="gz::sim::systems::JointStatePublisher">
+      <topic>joint_states</topic>
+    </plugin>
+    <plugin filename="libgz-sim-sensors-system.so" name="gz::sim::systems::Sensors">
+      <render_engine>ogre2</render_engine>
+    </plugin>
+  </gazebo>
 </robot>

File: urdf/waver.xacro (robot description, xacro)
@@ -1,11 +1,18 @@
 <?xml version="1.0"?>
 <robot name="waver" xmlns:xacro="http://www.ros.org/wiki/xacro">
+  <xacro:arg name="sim_control" default="gazebo" />
   <xacro:arg name="camera_type" default="raspi" />
   <xacro:include filename="$(find waver_description)/urdf/materials.xacro" />
   <xacro:include filename="$(find waver_description)/urdf/util.xacro" />
-  <!-- <xacro:include filename="$(find waver_description)/urdf/waver.trans.xacro" /> -->
-  <xacro:include filename="$(find waver_description)/urdf/waver.gazebo.xacro" />
   <xacro:include filename="$(find waver_description)/urdf/lidar.xacro" />
   <xacro:include filename="$(find waver_description)/urdf/imu.xacro" />
+  <!-- ************************** Simulation Control ************************** -->
+  <xacro:if value="${'$(arg sim_control)' == 'gazebo'}">
+    <xacro:include filename="$(find waver_description)/urdf/waver.gazebo.xacro" />
+  </xacro:if>
+  <xacro:if value="${'$(arg sim_control)' == 'ros2'}">
+    <xacro:include filename="$(find waver_description)/urdf/waver.control.xacro" />
+  </xacro:if>
+  <!-- ***************************** Camera Type ***************************** -->
   <xacro:if value="${'$(arg camera_type)' == 'raspi'}">
     <xacro:include filename="$(find waver_description)/urdf/camera.xacro" />
@@ -26,5 +33,5 @@
       <origin xyz="0 0 0" rpy="0 0 ${pi/2}" />
       <geometry>
-        <mesh filename="file:///$(find waver_description)/meshes/base_link.stl" scale="${scale}" />
+        <mesh filename="package://waver_description/meshes/base_link.stl" scale="${scale}" />
       </geometry>
       <xacro:dark_gray_material />
@@ -33,5 +40,5 @@
       <origin xyz="0 0 0" rpy="0 0 ${pi/2}" />
       <geometry>
-        <mesh filename="file:///$(find waver_description)/meshes/base_link.stl" scale="${scale}" />
+        <mesh filename="package://waver_description/meshes/base_link.stl" scale="${scale}" />
       </geometry>
     </collision>
@@ -47,5 +54,5 @@
       <origin xyz="0 0 0" rpy="0 0 ${pi/2}" />
       <geometry>
-        <mesh filename="file:///$(find waver_description)/meshes/top_shell_link.stl" scale="${scale}" />
+        <mesh filename="package://waver_description/meshes/top_shell_link.stl" scale="${scale}" />
       </geometry>
       <xacro:dark_gray_material />
@@ -54,19 +61,13 @@
       <origin xyz="0 0 0" rpy="0 0 ${pi/2}" />
       <geometry>
-        <mesh filename="file:///$(find waver_description)/meshes/top_shell_link.stl" scale="${scale}" />
+        <mesh filename="package://waver_description/meshes/top_shell_link.stl" scale="${scale}" />
       </geometry>
     </collision>
   </link>
   <link name="accessories_link">
-    <inertial>
-      <mass value="${mass_acces}" />
-      <origin xyz="${mass_center_acces}" rpy="0 0 ${pi/2}" />
-      <inertia ixx="1.284177729497181e-13" iyy="4.1792730400878273e-13" izz="4.1792732165684473e-13"
-        ixy="0.0" iyz="0.0" ixz="0.0" />
-    </inertial>
     <visual>
       <origin xyz="${position_acces}" rpy="0 0 ${pi/2}" />
       <geometry>
-        <mesh filename="file:///$(find waver_description)/meshes/accessories_link.stl" scale="${scale}" />
+        <mesh filename="package://waver_description/meshes/accessories_link.stl" scale="${scale}" />
       </geometry>
       <xacro:black_material />
@@ -75,49 +76,25 @@
       <origin xyz="${position_acces}" rpy="0 0 ${pi/2}" />
       <geometry>
-        <mesh filename="file:///$(find waver_description)/meshes/accessories_link.stl" scale="${scale}" />
+        <mesh filename="package://waver_description/meshes/accessories_link.stl" scale="${scale}" />
       </geometry>
     </collision>
   </link>
   <link name="accessories1_link">
-    <inertial>
-      <mass value="${mass_acces1}" />
-      <origin xyz="${mass_center_acces1}" rpy="0 0 ${pi/2}" />
-      <inertia ixx="8.4505377139432e-14" iyy="3.769648155305237e-13" izz="3.769601126710828e-13"
-        ixy="0.0" iyz="0.0" ixz="0.0" />
-    </inertial>
     <visual>
       <origin xyz="${position_acces1}" rpy="0 0 ${pi/2}" />
       <geometry>
-        <mesh filename="file:///$(find waver_description)/meshes/accessories1_link.stl" scale="${scale}" />
-      </geometry>
-      <xacro:black_material />
-    </visual>
-    <collision>
-      <origin xyz="${position_acces1}" rpy="0 0 ${pi/2}" />
-      <geometry>
-        <mesh filename="file:///$(find waver_description)/meshes/accessories1_link.stl" scale="${scale}" />
-      </geometry>
-    </collision>
+        <mesh filename="package://waver_description/meshes/accessories1_link.stl" scale="${scale}" />
+      </geometry>
+      <xacro:black_material />
+    </visual>
   </link>
   <link name="oled_screen_link">
-    <inertial>
-      <mass value="${mass_screen}" />
-      <origin xyz="${mass_center_screen}" rpy="0 0 ${pi/2}" />
-      <inertia ixx="2.2613546657562738e-14" iyy="1.821435448519393e-13" izz="1.9313666847229008e-13"
-        ixy="0.0" iyz="0.0" ixz="0.0" />
-    </inertial>
     <visual>
       <origin xyz="${position_screen}" rpy="0 0 ${pi/2}" />
       <geometry>
-        <mesh filename="file:///$(find waver_description)/meshes/oled_screen_link.stl" scale="${scale}" />
+        <mesh filename="package://waver_description/meshes/oled_screen_link.stl" scale="${scale}" />
       </geometry>
       <xacro:dark_blue_material />
     </visual>
-    <collision>
-      <origin xyz="${position_screen}" rpy="0 0 ${pi/2}" />
-      <geometry>
-        <mesh filename="file:///$(find waver_description)/meshes/oled_screen_link.stl" scale="${scale}" />
-      </geometry>
-    </collision>
   </link>
   <link name="wheel_back_left_link">
@@ -131,14 +108,13 @@
       <origin xyz="${position_wbl}" rpy="0 0 ${pi/2}" />
       <geometry>
-        <mesh filename="file:///$(find waver_description)/meshes/wheel_back_left_link.stl"
-          scale="${scale}" />
-      </geometry>
-      <xacro:black_material />
-    </visual>
-    <collision>
-      <origin xyz="${position_wbl}" rpy="0 0 ${pi/2}" />
-      <geometry>
-        <mesh filename="file:///$(find waver_description)/meshes/wheel_back_left_link.stl"
-          scale="${scale}" />
+        <mesh filename="package://waver_description/meshes/wheel_back_left_link.stl"
+          scale="${scale}" />
+      </geometry>
+      <xacro:black_material />
+    </visual>
+    <collision>
+      <origin xyz="0 0 0" rpy="${pi/2} 0 0" />
+      <geometry>
+        <cylinder radius="${wheel_radius}" length="${wheel_width}" />
       </geometry>
     </collision>
@@ -154,14 +130,13 @@
       <origin xyz="${position_wfl}" rpy="0 0 ${pi/2}" />
       <geometry>
-        <mesh filename="file:///$(find waver_description)/meshes/wheel_front_left_link.stl"
-          scale="${scale}" />
-      </geometry>
-      <xacro:black_material />
-    </visual>
-    <collision>
-      <origin xyz="${position_wfl}" rpy="0 0 ${pi/2}" />
-      <geometry>
-        <mesh filename="file:///$(find waver_description)/meshes/wheel_front_left_link.stl"
-          scale="${scale}" />
+        <mesh filename="package://waver_description/meshes/wheel_front_left_link.stl"
+          scale="${scale}" />
+      </geometry>
+      <xacro:black_material />
+    </visual>
+    <collision>
+      <origin xyz="0 0 0" rpy="${pi/2} 0 0" />
+      <geometry>
+        <cylinder radius="${wheel_radius}" length="${wheel_width}" />
       </geometry>
     </collision>
@@ -177,14 +152,13 @@
       <origin xyz="${position_wfr}" rpy="0 0 ${pi/2}" />
       <geometry>
-        <mesh filename="file:///$(find waver_description)/meshes/wheel_front_right_link.stl"
-          scale="${scale}" />
-      </geometry>
-      <xacro:black_material />
-    </visual>
-    <collision>
-      <origin xyz="${position_wfr}" rpy="0 0 ${pi/2}" />
-      <geometry>
-        <mesh filename="file:///$(find waver_description)/meshes/wheel_front_right_link.stl"
-          scale="${scale}" />
+        <mesh filename="package://waver_description/meshes/wheel_front_right_link.stl"
+          scale="${scale}" />
+      </geometry>
+      <xacro:black_material />
+    </visual>
+    <collision>
+      <origin xyz="0 0 0" rpy="${pi/2} 0 0" />
+      <geometry>
+        <cylinder radius="${wheel_radius}" length="${wheel_width}" />
       </geometry>
     </collision>
@@ -200,14 +174,13 @@
       <origin xyz="${position_wbr}" rpy="0 0 ${pi/2}" />
       <geometry>
-        <mesh filename="file:///$(find waver_description)/meshes/wheel_back_right_link.stl"
-          scale="${scale}" />
-      </geometry>
-      <xacro:black_material />
-    </visual>
-    <collision>
-      <origin xyz="${position_wbr}" rpy="0 0 ${pi/2}" />
-      <geometry>
-        <mesh filename="file:///$(find waver_description)/meshes/wheel_back_right_link.stl"
-          scale="${scale}" />
+        <mesh filename="package://waver_description/meshes/wheel_back_right_link.stl"
+          scale="${scale}" />
+      </geometry>
+      <xacro:black_material />
+    </visual>
+    <collision>
+      <origin xyz="0 0 0" rpy="${pi/2} 0 0" />
+      <geometry>
+        <cylinder radius="${wheel_radius}" length="${wheel_width}" />
       </geometry>
     </collision>
